File: tps709/tps709-breadboard-adapter.sch (KiCad schematic (older format))
At the start: 4 parts, among them J1 CONN_01X03, U1 TPS709xx

Commit message: Change tps709 adapter to use 0603 capacitors.
Parts:
- C1: footprint Capacitors_SMD:C_0805_HandSoldering -> Capacitors_SMD:C_0603_HandSoldering; MPN GRM21BR71E105KA99L -> GCM188R71E105KA64D; SPN 1828830 -> 2470425
- C2: footprint Capacitors_SMD:C_0805_HandSoldering -> Capacitors_SMD:C_0603_HandSoldering; MFR MURATA -> KEMET; MPN GRM21BR71E225KE11L -> C0603C225K8RACTU; SPN 2688538 -> 2491175
Changed lines of the file:
@@
 U 1 1 58D7C380
 P 3400 1300
-F 0 "U1" H 3600 1000 60  0000 C CNN
-F 1 "TPS709xx" H 3400 1600 60  0000 C CNN
-F 2 "TO_SOT_Packages_SMD:SOT-23-5_HandSoldering" H 3400 1300 60  0001 C CNN
-F 3 "http://www.ti.com/general/docs/lit/getliterature.tsp?genericPartNumber=TPS709&amp;&amp;fileType=pdf" H 3400 1300 60  0001 C CNN
-F 4 "TEXAS INSTRUMENTS" H -2050 -1150 50  0001 C CNN "MFR"
-F 5 "TPS70918DBVT" H -2050 -1150 50  0001 C CNN "MPN"
-F 6 "Farnell" H -2050 -1150 50  0001 C CNN "SPR"
-F 7 "2307954" H -2050 -1150 50  0001 C CNN "SPN"
+F 0 "U1" H 3600 1000 60 0000 C CNN
+F 1 "TPS709xx" H 3400 1600 60 0000 C CNN
+F 2 "TO_SOT_Packages_SMD:SOT-23-5_HandSoldering" H 3400 1300 60 0001 C CNN
+F 3 "http://www.ti.com/general/docs/lit/getliterature.tsp?genericPartNumber=TPS709&amp;&amp;fileType=pdf" H 3400 1300 60 0001 C CNN
+F 4 "TEXAS INSTRUMENTS" H -2050 -1150 50 0001 C CNN "MFR"
+F 5 "TPS70918DBVT" H -2050 -1150 50 0001 C CNN "MPN"
+F 6 "Farnell" H -2050 -1150 50 0001 C CNN "SPR"
+F 7 "2307954" H -2050 -1150 50 0001 C CNN "SPN"
+F 8 "" H 0 0 50 0001 C CNN "SPURL"
 	1    3400 1300
 	1    0    0    -1
@@
 U 1 1 58D7C3F5
 P 2650 1400
-F 0 "C1" H 2675 1500 50  0000 L CNN
-F 1 "1u" H 2675 1300 50  0000 L CNN
-F 2 "Capacitors_SMD:C_0805_HandSoldering" H 2688 1250 50  0001 C CNN
-F 3 "http://www.farnell.com/datasheets/2048734.pdf" H 2650 1400 50  0001 C CNN
-F 4 "GRM21BR71E105KA99L" H 2650 1400 60  0001 C CNN "MPN"
-F 5 "MURATA" H 2650 1400 60  0001 C CNN "MFR"
-F 6 "Farnell" H 2650 1400 60  0001 C CNN "SPR"
-F 7 "1828830" H 2650 1400 60  0001 C CNN "SPN"
+F 0 "C1" H 2675 1500 50 0000 L CNN
+F 1 "1u" H 2675 1300 50 0000 L CNN
+F 2 "Capacitors_SMD:C_0603_HandSoldering" H 2688 1250 50 0001 C CNN
+F 3 "http://www.farnell.com/datasheets/2048294.pdf" H 2650 1400 50 0001 C CNN
+F 4 "GCM188R71E105KA64D" H 2650 1400 60 0001 C CNN "MPN"
+F 5 "MURATA" H 2650 1400 60 0001 C CNN "MFR"
+F 6 "Farnell" H 2650 1400 60 0001 C CNN "SPR"
+F 7 "2470425" H 2650 1400 60 0001 C CNN "SPN"
+F 8 "" H 0 0 50 0001 C CNN "SPURL"
 	1    2650 1400
 	1    0    0    -1
@@
 U 1 1 58D7C462
 P 4150 1400
-F 0 "C2" H 4175 1500 50  0000 L CNN
-F 1 "2u2" H 4175 1300 50  0000 L CNN
-F 2 "Capacitors_SMD:C_0805_HandSoldering" H 4188 1250 50  0001 C CNN
-F 3 "http://www.farnell.com/datasheets/2189143.pdf" H 4150 1400 50  0001 C CNN
-F 4 "GRM21BR71E225KE11L" H 4150 1400 60  0001 C CNN "MPN"
-F 5 "MURATA" H 4150 1400 60  0001 C CNN "MFR"
-F 6 "Farnell" H 4150 1400 60  0001 C CNN "SPR"
-F 7 "2688538" H 4150 1400 60  0001 C CNN "SPN"
+F 0 "C2" H 4175 1500 50 0000 L CNN
+F 1 "2u2" H 4175 1300 50 0000 L CNN
+F 2 "Capacitors_SMD:C_0603_HandSoldering" H 4188 1250 50 0001 C CNN
+F 3 "http://www.farnell.com/datasheets/2205558.pdf" H 4150 1400 50 0001 C CNN
+F 4 "C0603C225K8RACTU" H 4150 1400 60 0001 C CNN "MPN"
+F 5 "KEMET" H 4150 1400 60 0001 C CNN "MFR"
+F 6 "Farnell" H 4150 1400 60 0001 C CNN "SPR"
+F 7 "2491175 " H 4150 1400 60 0001 C CNN "SPN"
+F 8 "" H 0 0 50 0001 C CNN "SPURL"
 	1    4150 1400
 	1    0    0    -1
@@
 U 1 1 58D7C54C
 P 2650 1650
-F 0 "#PWR01" H 2650 1400 50  0001 C CNN
-F 1 "GND" H 2650 1500 50  0000 C CNN
-F 2 "" H 2650 1650 50  0001 C CNN
-F 3 "" H 2650 1650 50  0001 C CNN
+F 0 "#PWR01" H 2650 1400 50 0001 C CNN
+F 1 "GND" H 2650 1500 50 0000 C CNN
+F 2 "" H 2650 1650 50 0001 C CNN
+F 3 "" H 2650 1650 50 0001 C CNN
 	1    2650 1650
 	1    0    0    -1
@@
 U 1 1 58D7C567
 P 2850 1650
-F 0 "#PWR02" H 2850 1400 50  0001 C CNN
-F 1 "GND" H 2850 1500 50  0000 C CNN
-F 2 "" H 2850 1650 50  0001 C CNN
-F 3 "" H 2850 1650 50  0001 C CNN
+F 0 "#PWR02" H 2850 1400 50 0001 C CNN
+F 1 "GND" H 2850 1500 50 0000 C CNN
+F 2 "" H 2850 1650 50 0001 C CNN
+F 3 "" H 2850 1650 50 0001 C CNN
 	1    2850 1650
 	1    0    0    -1
@@
 U 1 1 58D7C57B
 P 4150 1650
-F 0 "#PWR03" H 4150 1400 50  0001 C CNN
-F 1 "GND" H 4150 1500 50  0000 C CNN
-F 2 "" H 4150 1650 50  0001 C CNN
-F 3 "" H 4150 1650 50  0001 C CNN
+F 0 "#PWR03" H 4150 1400 50 0001 C CNN
+F 1 "GND" H 4150 1500 50 0000 C CNN
+F 2 "" H 4150 1650 50 0001 C CNN
+F 3 "" H 4150 1650 50 0001 C CNN
 	1    4150 1650
 	1    0    0    -1
@@
 U 1 1 58D82A52
 P 1800 1400
-F 0 "J1" H 1800 1600 50  0000 C CNN
-F 1 "CONN_01X03" V 1900 1400 50  0000 C CNN
-F 2 "Pin_Headers:Pin_Header_Straight_1x03_Pitch2.54mm" H 1800 1400 50  0001 C CNN
-F 3 "http://www.farnell.com/datasheets/1697160.pdf" H 1800 1400 50  0001 C CNN
-F 4 "HARWIN" H -2050 -1150 50  0001 C CNN "MFR"
-F 5 "M20-9990345" H -2050 -1150 50  0001 C CNN "MPN"
-F 6 "Farnell" H -2050 -1150 50  0001 C CNN "SPR"
-F 7 "1022248" H -2050 -1150 50  0001 C CNN "SPN"
+F 0 "J1" H 1800 1600 50 0000 C CNN
+F 1 "CONN_01X03" V 1900 1400 50 0000 C CNN
+F 2 "Pin_Headers:Pin_Header_Straight_1x03_Pitch2.54mm" H 1800 1400 50 0001 C CNN
+F 3 "http://www.farnell.com/datasheets/1697160.pdf" H 1800 1400 50 0001 C CNN
+F 4 "HARWIN" H -2050 -1150 50 0001 C CNN "MFR"
+F 5 "M20-9990345" H -2050 -1150 50 0001 C CNN "MPN"
+F 6 "Farnell" H -2050 -1150 50 0001 C CNN "SPR"
+F 7 "1022248" H -2050 -1150 50 0001 C CNN "SPN"
+F 8 "" H 0 0 50 0001 C CNN "SPURL"
 	1    1800 1400
 	-1   0    0    -1
